File: MCU Datalogger.kicad_sch (KiCad schematic)
At the start: 25 parts, among them U1 24LC1025, U2 DS1337S+, U3 24LC1025, U4 ATMEGA328P-AU, Y1 32.768 KHz, Y2 16 MHz

Commit message: UPdates
Other:
- note added: "Something here"
Changed lines of the file:
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@@
+    (effects (font (size 1.27 1.27)) (justify left bottom))
+  )
+  (text "Something here\n" (at 199.39 115.57 0)
     (effects (font (size 1.27 1.27)) (justify left bottom))
   )
