File: connectors.kicad_sch (KiCad schematic)
At the start: 4 parts, among them J1 Conn_01x04_Male, J2 Conn_01x09_Male, J3 Conn_01x04_Male, J4 Conn_02x03_Odd_Even

Commit message: Test
Other:
- company: (none) -> COMPANY
- title: (none) -> ${project_name}
